File: electronics/halo_rev_a/out/halo_rev_a.kicad_sch (KiCad schematic)
At the start: 51 parts, among them J1 TC2030, J2 UWB stub, U1 nRF54L10-QFAA-R7, U2 LIS2DW12TR, U3 GD25LQ32E 32Mbit, X1 32.768kHz, X2 32MHz

Commit message: sim (lane B1): the sounder measured, and R9 earns its BOM line - PASS
D11a deletes the class-D amplifier and drives a bare piezo bender straight
from two SoC pins. research/05 section 11.6 argues on arithmetic that this
costs nothing, and ends by calling itself 'derived arithmetic from the
datasheet capacitance class, not a measurement'. This is the measurement of
the electrical half. Seven circuits, VERDICT PASS.

D11a's CENTRAL CLAIM HOLDS. Two GPIO in anti-phase put 3.98 V peak to peak
across the bender from a 2.0 V end-of-life cell - the same 2 x VDD a
bridge-tied class-D would give, from no amplifier at all.

R9 IS LOAD-BEARING, and the schematic's stated reason for it was wrong. With
a low-loss 40 nF bender the peak pin current is 32.0 mA with R9 removed and
17.8 mA with it fitted: a 44 percent cut, and the difference between
exceeding a 25 mA ceiling and clearing it. The schematic said '100 R holds
the peak near 30 mA', which had the right magnitude and the wrong side of
it; that note now carries the measured pair.

Rail while sounding: no measurable droop. RMS draw is 1.9 to 4.6 mA against
40 uF of bulk, so the alert does not brown out the radio that has to keep
advertising through it.

TWO THINGS THIS STUDY GOT WRONG FIRST, both caught by its own asserts.

The first version measured pp_of('bend_p') - the voltage at ONE END of the
bender relative to ground - and reported 2.0 V where the differential swing
is 4.0 V. It graded the wrong quantity and failed an assert that was
actually satisfied. A behavioural source now makes the difference a node the
measurement can see. An assert that passes without checking what matters is
worse than a failure; this one failed, which is how it was found.

The second was the bender's series loss. 500 ohm is lane G's figure via
design.py, read here as a series loss resistance - but |Z| of 25 nF at 4 kHz
is 1592 ohm, so 500 ohm may be the motional resistance AT resonance, a
different element entirely. At 500 ohm the bender's ow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
Parts:
- R9: Note series damping on one leg. A bender is a near-pure capacita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 -> series damping on one leg, and it EARNS ITS PLACE - measure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
Other:
- note added: "ACCEL"
- note added: "BATTERY"
- note added: "CLOCKS"
- note added: "DEBUG"
- note added: "FLASH"
- note added: "NFC"
- note added: "POWER"
- note added: "RF"
- note added: "SOC"
- note added: "SOUNDER"
- note added: "UWB"
- moved on the sheet: AE1, AE2, BT1, C1, C10, C11, C12, C13, C14, C15, C16, C17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

Commit message: electronics (lane B1): flash deleted as out-of-spec, test access designed in, antenna re-sized from a measurement
THE FLASH WAS A REAL DEFECT AND IT IS GONE. U3 was a GD25LQ32EEIGR sitting
on VDD, which on this board is a raw CR2032 with no regulator anywhere. That
part's supply range is 1.65 to 2.0 V and a fresh coin cell is 3.0 V, so it
was out of specification from the first second - the kind of fault that
half-works on a bench and fails in a field. Caught by the production test
lane reading the sheet.

Fitting a regulator was the other way out and it is what the real AirTag
does (a TPS62746 buck plus an FPF2487 load switch, SPEC.md section 3). It
would have cost a part, an inductor, a rail, a test and board area this disc
does not have, and bought nothing: the SoC, the accelerometer and the bender
all span the whole cell curve unaided. research/05 section 3.7 and
spec/bom-candidates.json already recommended omitting the flash, and the
firmware lane has since measured the whole firmware at 13,164 bytes - 1.27
percent of the nRF54L10's own 1 MB. So it is deleted: a part, a rail
problem, two pull-ups, nine joints and a production test. If revision B ever
wants external firmware staging the part is a wide-range low-power NOR such
as the Macronix MX25R, specified 1.65 to 3.6 V, which is the range a coin
cell actually presents.

TEST ACCESS IS DESIGNED IN. Eleven probe lands, and VDD and GND each get a
FORCE and a SENSE pad rather than one pad each - sleep current here is
single-digit microamps and a two-wire reading measures the probe, while two
probes in one battery pad is a two-wire measurement wearing a four-wire
name. Plus both piezo nets, which otherwise terminate on the shell; the
cell-removal sense node; the I2C bus; both NFC pins; and two fiducials.
IPC-A-610 CLASS 2 is recorded on the sheet, because the AOI recipe is built
from it and nobody had chosen one.

THEY ARE PLACED BY SEARCH, NOT BY HAND. Hand-placing thirteen things into a
full board produced eight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
Parts:
- removed R3, R4: 100k, Resistor_SMD:R_0201_0603Metric, symbol Device:R
- removed U3: GD25LQ32E 32Mbit, Package_SON:Winbond_USON-8-1EP_3x2mm_P0.5mm_EP0.2x1.6mm, symbol Memory_Flash:W25Q32JVSS
- added FID1, FID2: FIDUCIAL, Fiducial:Fiducial_0.5mm_Mask1mm, symbol Mechanical:Fiducial
- added TP1, TP10, TP11, TP2, TP3, TP4, TP5, TP6, TP7, TP8, TP9: TP, halo:HALO_TP_D0.8, symbol Connector:TestPoint
- C24, C25: value 130pF -> 1.1nF; LCSC C1571 -> C1546; MPN CL03C131JB3NNNC -> 0201 C0G 1.1nF; Manufacturer Samsung -> TBC; Note NFC tuning, PLACEHOLDER (X-2). 130 pF is Nordic's NFCT chap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 -> NFC tuning, MEASURED not assumed: ce-rf gives the 2-turn co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; Price@1k $0.0029 -> TBC; Stock in stock -> TBC
- J2: footprint halo:HALO_CASTELLATED_1x08_P1.00 -> halo:HALO_UWB_LANDS_1x08_P1.00; Note 8 CASTELLATED HALF-VIAS on the board edge, reserving the ha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 -> 8 SMD LANDS just inboard of the board edge, reserving the h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
Connections:
- net GND: now also TP3.1, TP4.1
- net I2C_SCL: now also TP9.1
- net I2C_SDA: now also TP8.1
- net NFC1: now also TP10.1
- net NFC2: now also TP11.1
- net PIEZO_N: now also TP6.1
- net PIEZO_P: now also TP5.1
- net VBAT_SNS: now also TP7.1
- net VDD: now also TP1.1, TP2.1
- net FLASH_CS: no longer names the net of U1.16 (P2.05/CS)
- no-connect marks 11 -> 12
Other:
- note added: "IPC-A-610 ACCEPTANCE CLASS 2. Class 3 is for equipment whose failure cannot be tolerated - life support, avionics - and halo is not that. Class 1 is general consumer electronics where cosmetics do not matter, and a product with a DULT safety obligation and a user-replaceable cell is not that either. The AOI recipe is built from this line, so it is recorded here rather than left for the factory to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"
- note added: "TEST"
- note added: "TEST ACCESS (block 10): TP1/TP2 are VDD FORCE and SENSE and TP3/TP4 are GND FORCE and SENSE - four wires, because sleep current here is single-digit microamps and a two-wire reading measures the probe. FID1/FID2 are ASYMMETRIC: a 26 mm circle has no datum and without them every pad position is a guess."
- note added: "THERE IS NO SPI NOR FLASH. The GD25LQ32E first drawn here is a 1.65-2.0 V part and this board's only rail is a raw 3.0 V coin cell. Block 6 carries the argument; the firmware is 13,164 bytes, 1.27 % of the SoC's own 1 MB."
- note removed: "FLASH"
- moved on the sheet: AE1, AE2, BT1, C10, C11, C12, C13, C14, C15, C16, C17, C18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

Commit message: fab (lane B1): the factory package - gerbers with geometry, a BOM with order codes, ERC 0/0
ERC PASS, 0 errors AND 0 WARNINGS. The 13 warnings before this were one
cause: this machine has no global KiCad footprint table, because KiCad has
never been opened interactively here, so without a project table ERC cannot
resolve a footprint and reports one warning per part. The project now writes
its own listing all 155 KiCad libraries plus halo's, which also makes the
handoff self-contained. It is written at the END of the pipeline because
bin/sch build writes its own 8-library version over anything earlier - an
attempt to write it from the schematic was silently discarded.

THE GERBERS ARE VERIFIED, NOT ASSUMED. The factory lane warned that gerber
export had been failing silently for everyone - a flag that does not exist
in KiCad 10 while the pipeline reported success - so these were opened
rather than trusted: F_Cu carries 3265 draw commands and Edge_Cuts 720. 13
files in the zip, layer check PASS against JLCPCB's published naming table,
plus two Excellon drills and a drill map.

THE BOM CARRIES ORDER CODES NOW, and it did not an hour ago. Two silent
failures stacked. First, the field was named 'LCSC' and ce-fab looks for
'LCSC Part #' and five other spellings - a plain 'LCSC' is in none of them.
Second, and worse, Board.place() puts a land pattern down without the part's
value or its fields, because those live on the schematic; fab jlc reads the
.kicad_pcb, so every order code was on the sheet and NOT ONE reached the
bill of materials. The board now imports the schematic and copies 61 values
and 324 fields across. 24 BOM lines with real codes; the six parts with no
code are AE1 and AE2, which are etched copper, and C14-C17, which are not
fitted. Those are correct answers, not gaps.

THE RULE THAT FIRES IS NOW THE RULE THE REPORT NAMES - the other trap the
factory lane flagged. The DRC had been running against KiCad's 0.5 mm
default board-edge clearance while this board'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
Parts:
- BT1: LCSC C7498149 -> (none); LCSC Part # (none) -> C7498149
- C1, C2, C24, C25, C3, C4: LCSC C1546 -> (none); LCSC Part # (none) -> C1546
- C10, C11, C12, C9: LCSC C15525 -> (none); LCSC Part # (none) -> C15525
- C13: LCSC C1523 -> (none); LCSC Part # (none) -> C1523
- C18, C19, C20, C21, C22, C23: LCSC C1568 -> (none); LCSC Part # (none) -> C1568
- C5, C6, C7, C8: LCSC C2827888 -> (none); LCSC Part # (none) -> C2827888
- FID1, FID2: LCSC n/a - bare copper -> (none); LCSC Part # (none) -> n/a
- J1: LCSC n/a - pads only, no part -> (none); LCSC Part # (none) -> n/a
- J2: LCSC n/a - castellations, no part -> (none); LCSC Part # (none) -> n/a
- L1: LCSC C1046 -> (none); LCSC Part # (none) -> C1046
- L10, R9: LCSC C25076 -> (none); LCSC Part # (none) -> C25076
- L2, L3, L4: LCSC C1046539 -> (none); LCSC Part # (none) -> C1046539
- LS1: LCSC NOT IN CATALOGUE -> (none); LCSC Part # (none) -> NOT IN CATALOGUE
- R1, R2: LCSC C25765 -> (none); LCSC Part # (none) -> C25765
- R10, R5, R6, R7, R8: LCSC C25744 -> (none); LCSC Part # (none) -> C25744
- TP1, TP10, TP11, TP2, TP3, TP4, TP5, TP6, TP7, TP8, TP9: LCSC n/a - a pad, not a part -> (none); LCSC Part # (none) -> n/a
- U1: LCSC C44800139 -> (none); LCSC Part # (none) -> C44800139
- U2: LCSC C189624 -> (none); LCSC Part # (none) -> C189624
- X1: LCSC C620155 -> (none); LCSC Part # (none) -> C32346; MPN X321532768KGD2SI -> FC-135 32.768kHz; Manufacturer Yangxing Tech -> Epson; Note CL 12.5 pF, +/-20 ppm. 3.2x1.5x0.9 mm - 0.9 mm TALL, which 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 -> Epson 32.768 kHz. CHANGED from X321532768KGD2SI (C620155) o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; Price@1k $0.1347 -> $0.1375; Stock in stock -> 444,985
- X2: LCSC C843260 -> (none); LCSC Part # (none) -> C843260
Changed lines of the file:
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@@
 			)
 		)
-		(property "LCSC" "C44800139"
+		(property "LCSC Part #" "C44800139"
 			(at 40.64 102.87 0)
 			(effects
@@
 			)
 		)
-		(property "LCSC" "C1546"
+		(property "LCSC Part #" "C1546"
 			(at 88.9 39.37 0)
 			(effects
@@
 			)
 		)
-		(property "LCSC" "C1546"
+		(property "LCSC Part #" "C1546"
 			(at 88.9 69.85 0)
 			(effects
@@
 			)
 		)
-		(property "LCSC" "C1546"
+		(property "LCSC Part #" "C1546"
 			(at 88.9 101.6 0)
 			(effects
@@
 			)
 		)
-		(property "LCSC" "C1546"
+		(property "LCSC Part #" "C1546"
 			(at 88.9 132.08 0)
 			(effects
@@
 			)
 		)
-		(property "LCSC" "C1046"
+		(property "LCSC Part #" "C1046"
 			(at 87.63 163.83 0)
 			(effects
@@
 			)
 		)
-		(property "LCSC" "C2827888"
+		(property "LCSC Part #" "C2827888"
 			(at 118.11 39.37 0)
 			(effects
@@
 			)
 		)
-		(property "LCSC" "C2827888"
+		(property "LCSC Part #" "C2827888"
 			(at 118.11 69.85 0)
 			(effects
@@
 			)
 		)
-		(property "LCSC" "C2827888"
+		(property "LCSC Part #" "C2827888"
 			(at 118.11 101.6 0)
 			(effects
@@
 			)
 		)
-		(property "LCSC" "C2827888"
+		(property "LCSC Part #" "C2827888"
 			(at 118.11 132.08 0)
 			(effects
@@
 			)
 		)
-		(property "LCSC" "C7498149"
+		(property "LCSC Part #" "C7498149"
 			(at 171.45 39.37 0)
 			(effects
@@
 			)
 		)
-		(property "LCSC" "C15525"
+		(property "LCSC Part #" "C15525"
 			(at 148.59 69.85 0)
 			(effects
@@
 			)
 		)
-		(property "LCSC" "C15525"
+		(property "LCSC Part #" "C15525"
 			(at 148.59 101.6 0)
 			(effects
@@
 			)
 		)
-		(property "LCSC" "C15525"
+		(property "LCSC Part #" "C15525"
 			(at 148.59 132.08 0)
 			(effects
@@
 			)
 		)
-		(property "LCSC" "C15525"
+		(property "LCSC Part #" "C15525"
 			(at 148.59 163.83 0)
 			(effects
@@
 			)
 		)
-		(property "LCSC" "C25765"
+		(property "LCSC Part #" "C25765"
 			(at 231.14 39.37 0)
 			(effects
@@
 			)
 		)
-		(property "LCSC" "C25765"
+		(property "LCSC Part #" "C25765"
 			(at 228.6 69.85 0)
 			(effects
@@
 			)
 		)
-		(property "LCSC" "C1523"
+		(property "LCSC Part #" "C1523"
 			(at 228.6 101.6 0)
 			(effects
@@
 			)
 		)
-		(property "LCSC" "C620155"
+		(property "LCSC Part #" "C32346"
 			(at 269.24 36.83 0)
 			(effects
@@
 			)
 		)
-		(property "MPN" "X321532768KGD2SI"
+		(property "MPN" "FC-135 32.768kHz"
 			(at 269.24 36.83 0)
 			(effects
@@
 			)
 		)
-		(property "Manufacturer" "Yangxing Tech"
+		(property "Manufacturer" "Epson"
 			(at 269.24 36.83 0)
 			(effects
@@
 			)
 		)
-		(property "Note" "CL 12.5 pF, +/-20 ppm. 3.2x1.5x0.9 mm - 0.9 mm TALL, which X-5's height delta also binds. A 2012 part would fit; none was priced by lane E."
+		(property "Note" "Epson 32.768 kHz. CHANGED from X321532768KGD2SI (C620155) on the factory lane's find: C32346 is a JLCPCB BASIC part with 444,985 in stock at $0.1375/100, so it avoids the $3.07 extended-part feeder fee as well as being deeper stock. OPEN: its package is assumed to be the 3215 land pattern drawn here and that has NOT been confirmed against Epson's drawing - confirm before ordering. Still 0.9 mm tall, which X-5's height delta binds."
 			(at 269.24 36.83 0)
 			(effects
@@
 			)
 		)
-		(property "Price@1k" "$0.1347"
+		(property "Price@1k" "$0.1375"
 			(at 269.24 36.83 0)
 			(effects
@@
 			)
 		)
-		(property "Stock" "in stock"
+		(property "Stock" "444,985"
 			(at 269.24 36.83 0)
 			(effects
@@
 			)
 		)
-		(property "LCSC" "C843260"
+		(property "LCSC Part #" "C843260"
 			(at 269.24 68.58 0)
 			(effects
@@
 			)
 		)
-		(property "LCSC" "C1046539"
+		(property "LCSC Part #" "C1046539"
 			(at 330.2 69.85 0)
 			(effects
@@
 			)
 		)
-		(property "LCSC" "C1046539"
+		(property "LCSC Part #" "C1046539"
 			(at 327.66 101.6 0)
 			(effects
@@
 			)
 		)
-		(property "LCSC" "C1046539"
+		(property "LCSC Part #" "C1046539"
 			(at 328.93 132.08 0)
 			(effects
@@
 			)
 		)
-		(property "LCSC" "C1568"
+		(property "LCSC Part #" "C1568"
 			(at 330.2 163.83 0)
 			(effects
@@
 			)
 		)
-		(property "LCSC" "C1568"
+		(property "LCSC Part #" "C1568"
 			(at 368.3 39.37 0)
 			(effects
@@
 			)
 		)
-		(property "LCSC" "C1568"
+		(property "LCSC Part #" "C1568"
 			(at 369.57 69.85 0)
 			(effects
@@
 			)
 		)
-		(property "LCSC" "C1568"
+		(property "LCSC Part #" "C1568"
 			(at 370.84 101.6 0)
 			(effects
@@
 			)
 		)
-		(property "LCSC" "C1568"
+		(property "LCSC Part #" "C1568"
 			(at 369.57 132.08 0)
 			(effects
@@
 			)
 		)
-		(property "LCSC" "C25076"
+		(property "LCSC Part #" "C25076"
 			(at 370.84 163.83 0)
 			(effects
@@
 			)
 		)
-		(property "LCSC" "C1568"
+		(property "LCSC Part #" "C1568"
 			(at 408.94 39.37 0)
 			(effects
@@
 			)
 		)
-		(property "LCSC" "C1546"
+		(property "LCSC Part #" "C1546"
 			(at 444.5 71.12 0)
 			(effects
@@
 			)
 		)
-		(property "LCSC" "C1546"
+		(property "LCSC Part #" "C1546"
 			(at 444.5 102.87 0)
 			(effects
@@
 			)
 		)
-		(property "LCSC" "C189624"
+		(property "LCSC Part #" "C189624"
 			(at 495.3 54.61 0)
 			(effects
@@
 			)
 		)
-		(property "LCSC" "C25744"
+		(property "LCSC Part #" "C25744"
 			(at 480.06 85.09 0)
 			(effects
@@
 			)
 		)
-		(property "LCSC" "C25744"
+		(property "LCSC Part #" "C25744"
 			(at 481.33 116.84 0)
 			(effects
@@
 			)
 		)
-		(property "LCSC" "C25744"
+		(property "LCSC Part #" "C25744"
 			(at 481.33 147.32 0)
 			(effects
@@
 			)
 		)
-		(property "LCSC" "C25744"
+		(property "LCSC Part #" "C25744"
 			(at 481.33 179.07 0)
 			(effects
@@
 			)
 		)
-		(property "LCSC" "NOT IN CATALOGUE"
+		(property "LCSC Part #" "NOT IN CATALOGUE"
 			(at 548.64 36.83 0)
 			(effects
@@
 			)
 		)
-		(property "LCSC" "C25076"
+		(property "LCSC Part #" "C25076"
 			(at 547.37 68.58 0)
 			(effects
@@
 			)
 		)
-		(property "LCSC" "n/a - pads only, no part"
+		(property "LCSC Part #" "n/a"
 			(at 27.94 233.68 0)
 			(effects
@@
 			)
 		)
-		(property "LCSC" "C25744"
+		(property "LCSC Part #" "C25744"
 			(at 24.13 264.16 0)
 			(effects
@@
 			)
 		)
-		(property "LCSC" "n/a - castellations, no part"
+		(property "LCSC Part #" "n/a"
 			(at 74.93 233.68 0)
 			(effects
@@
 			)
 		)
-		(property "LCSC" "n/a - a pad, not a part"
+		(property "LCSC Part #" "n/a"
 			(at 106.68 217.17 0)
 			(effects
@@
 			)
 		)
-		(property "LCSC" "n/a - a pad, not a part"
+		(property "LCSC Part #" "n/a"
 			(at 106.68 243.84 0)
 			(effects
@@
 			)
 		)
-		(property "LCSC" "n/a - a pad, not a part"
+		(property "LCSC Part #" "n/a"
 			(at 106.68 270.51 0)
 			(effects
@@
 			)
 		)
-		(property "LCSC" "n/a - a pad, not a part"
+		(property "LCSC Part #" "n/a"
 			(at 106.68 297.18 0)
 			(effects
@@
 			)
 		)
-		(property "LCSC" "n/a - a pad, not a part"
+		(property "LCSC Part #" "n/a"
 			(at 110.49 323.85 0)
 			(effects
@@
 			)
 		)
-		(property "LCSC" "n/a - a pad, not a part"
+		(property "LCSC Part #" "n/a"
 			(at 110.49 350.52 0)
 			(effects
@@
 			)
 		)
-		(property "LCSC" "n/a - a pad, not a part"
+		(property "LCSC Part #" "n/a"
 			(at 144.78 217.17 0)
 			(effects
@@
 			)
 		)
-		(property "LCSC" "n/a - a pad, not a part"
+		(property "LCSC Part #" "n/a"
 			(at 143.51 243.84 0)
 			(effects
@@
 			)
 		)
-		(property "LCSC" "n/a - a pad, not a part"
+		(property "LCSC Part #" "n/a"
 			(at 143.51 270.51 0)
 			(effects
@@
 			)
 		)
-		(property "LCSC" "n/a - a pad, not a part"
+		(property "LCSC Part #" "n/a"
 			(at 140.97 297.18 0)
 			(effects
@@
 			)
 		)
-		(property "LCSC" "n/a - a pad, not a part"
+		(property "LCSC Part #" "n/a"
 			(at 140.97 323.85 0)
 			(effects
@@
 			)
 		)
-		(property "LCSC" "n/a - bare copper"
+		(property "LCSC Part #" "n/a"
 			(at 135.89 346.71 0)
 			(effects
@@
 			)
 		)
-		(property "LCSC" "n/a - bare copper"
+		(property "LCSC Part #" "n/a"
 			(at 172.72 213.36 0)
 			(effects
