File: electronics/halo_rev_a/out/halo_rev_a.kicad_sch (KiCad schematic)
At the start: 61 parts, among them J1 TC2030, J2 UWB stub, U1 nRF54L10-QFAA-R7, U2 LIS2DW12TR, X1 32.768kHz, X2 32MHz

Commit message: B1: the crystal was out of spec, 1.1 nF does not exist, and the net tie was three times too wide
THE FOUR CHANGES FROM SOURCING AND VERIFICATION, ALL FOUR LANDED.

1. X1 IS THE WRONG CRYSTAL AND WOULD NOT HAVE STARTED. C32346 (Q13FC13500004)
   is CL = 12.5 pF, chosen on price and stock, and D-3 deletes the external
   load capacitors — so the entire load is the nRF54L's on-die caps. Nordic's
   datasheet 4503_018 v1.0 (Sept 2025) refuses 12.5 pF twice:
     * Sec 5.5.2 — OSCILLATORS.XOSC32KI.INTCAP holds 3-18 pF in 0.65 pF steps,
       and CL = (C_INT + C_pcb)/2, so the ceiling is about (18+2)/2 = 10 pF.
       12.5 pF needs C_INT ~ 23 pF: 5 pF above the hardware maximum.
     * Sec 11.9.2 — CL_LFXO min 6 pF, MAX 9 pF, at the part level, whether the
       capacitors are internal or external.
   Nordic's own reference BOM (Sec 10.3) is a CL 9 pF crystal with NO external
   load capacitors. X1 is now C95361 (Q13FC13500049), the same Epson FC-135
   body at CL 6 pF, 134,310 in stock. This is the failure the brief described:
   the crystal does not start and the board looks simply dead.

2. 1.1 nF DOES NOT EXIST, SO THE COIL MOVES INSTEAD. No 1.1 nF capacitor is
   made in 0201 in any dielectric, none in 0402, and the smallest anywhere is
   0603 — three sizes too big. C24/C25 are 1.0 nF C0G (C161371, 139,150 in
   stock) and the tank is retuned in copper, which is free: series C
   554.6 -> 500 pF, so L must rise by 554.6/500 = 1.1092, from ce-rf's
   measured 0.2449 uH to a TARGET of 0.2716 uH. footprints.py NFC_TURNS is
   DERIVED from that ratio — 2.000 -> 2.1062 turns on N-squared scaling —
   moving the innermost turn from R10.150 to R10.118, copper edge R10.043
   against the Ø20.0 cell can at R10.000. THE INDUCTANCE AT THIS LENGTH IS NOT
   MEASURED: N-squared is Wheeler's first term and ce-rf owns the solve, so
   the resonant frequency is CANNOT DETERMINE until that run exists.

3. DNP REACHES THE BOARD. The field-carry loop copied values and fields and
   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
Parts:
- BT1: LCSC Part # C7498149 -> NO ORDER CODE - NOT AN SMT LINE; Note THE FOOTPRINT IS halo's OWN, drawn by the layout: three pad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 -> THE CELL IS BOUGHT, THE HOLDER IS NOT: no part is fitted on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; Price@1k $0.39 -> (none); Priced 2026-09-03 -> (none); Stock in stock -> (none)
- C1: LCSC Part # C1546 -> C5142565; MPN CL03A104KA3NNNC -> TCC0201X5R104K100ZT; Manufacturer Samsung -> CCTC; Note 0201 X7R 16V, at VDD pin 10 -> 0201 X5R 10V, at VDD pin 10. Code re-verified 2026-09-05: C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; Price@1k $0.0029 -> $0.0005
- C13: LCSC Part # C1523 -> C76922; MPN CL03C101JB3NNNC -> GRM0335C1H101JA01D; Manufacturer Samsung -> muRata; Note settles the divider inside the ADC's acquisition window; also sets the ~0.24 ms collapse time when the cell leaves -> settles the divider inside the ADC's acquisition window; also sets the ~0.24 ms collapse time when the cell leaves. Code re-verified 2026-09-05: C1523 is a 1 nF 0402 (S1).; Price@1k $0.0029 -> $0.0033
- C18: LCSC Part # C1568 -> C435397; MPN GJM0335C1E1R5WB01 -> GJM0335C1E1R5WB01D; Note 0201 NP0 high-Q. LAYOUT RULE: its ground connects ONLY to pin 32 (VSS_PA), on the top layer. Nordic's words, Figure 175. -> 0201 NP0 high-Q. LAYOUT RULE: its ground connects ONLY to pin 32 (VSS_PA), on the top layer. Nordic's words, Figure 175. Code re-verified 2026-09-05 (S1).; Price@1k $0.0091 -> $0.0262
- C19: LCSC Part # C1568 -> C668326; MPN GJM0335C1E1R5WB01 -> GJM0335C1E2R0WB01D; Note 0201 NP0. LAYOUT RULE: its ground MUST be isolated from every ground layer except the bottom. Nordic's words, Figure 175. -> 0201 NP0. LAYOUT RULE: its ground MUST be isolated from every ground layer except the bottom. Nordic's words, Figure 175. Code re-verified 2026-09-05 (S1).; Price@1k $0.0091 -> $0.0262
- C2: LCSC Part # C1546 -> C5142565; MPN CL03A104KA3NNNC -> TCC0201X5R104K100ZT; Manufacturer Samsung -> CCTC; Note 0201 X7R 16V, at VDD pin 22 -> 0201 X5R 10V, at VDD pin 22. Code re-verified 2026-09-05: C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; Price@1k $0.0029 -> $0.0005
- C20: LCSC Part # C1568 -> C237424; MPN GJM0335C1ER50WB01 -> GJM0335C1HR50WB01D; Note PI SHUNT, source side. PLACEHOLDER - value comes from ce-rf S11 on the real copper. -> PI SHUNT, source side. PLACEHOLDER - value comes from ce-rf S11 on the real copper. Code re-verified 2026-09-05: C1568 is 4 pF 0402 (S1).; Price@1k $0.0091 -> $0.0223
- C21: LCSC Part # C1568 -> C237424; MPN GJM0335C1ER50WB01 -> GJM0335C1HR50WB01D; Price@1k $0.0091 -> $0.0223
- C22: LCSC Part # C1568 -> C3904589; MPN GJM0335C1E1R5WB01 -> GJM0335C1HR30WB01D; Note 0201 C0G, series trim into the pi -> 0201 C0G, series trim into the pi Code re-verified 2026-09-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; Price@1k $0.0091 -> $0.0262
- C23: LCSC Part # C1568 -> C1852416; MPN GJM0335C1E1R5WB01 -> GJM0335C1E3R9WB01D; Note 0201 C0G - Table 82 lists it, Figure 175's extraction does not place its node. Wired as a shunt at ANT. CANNOT DETERMINE. -> 0201 C0G - Table 82 lists it, Figure 175's extraction does not place its node. Wired as a shunt at ANT. CANNOT DETERMINE. Code re-verified 2026-09-05 (S1).; Price@1k $0.0091 -> $0.0262
- C24, C25: value 1.1nF -> 1.0nF; LCSC Part # C1546 -> C161371; MPN 0201 C0G 1.1nF -> GRM0335C1E102JA01D; Manufacturer TBC -> muRata; Note NFC tuning, MEASURED not assumed: ce-rf gives the 2-turn co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 -> NFC tuning. 1.109 nF was the arithmetic; 1.0 nF is what exi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; Stock TBC -> 139,150
- C3: LCSC Part # C1546 -> C5142565; MPN CL03A104KA3NNNC -> TCC0201X5R104K100ZT; Manufacturer Samsung -> CCTC; Note 0201 X7R 16V, at VDD pin 36 -> 0201 X5R 10V, at VDD pin 36. Code re-verified 2026-09-05: C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; Price@1k $0.0029 -> $0.0005
- C4: LCSC Part # C1546 -> C5142565; MPN CL03A104KA3NNNC -> TCC0201X5R104K100ZT; Manufacturer Samsung -> CCTC; Note 0201 X7R 16V, at VDD pins 47/48 -> 0201 X5R 10V, at VDD pins 47/48. Code re-verified 2026-09-0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; Price@1k $0.0029 -> $0.0005
- C5: LCSC Part # C2827888 -> C335106; MPN CL03A225MQ3CSNC -> GRM033R61A225KE47D; Manufacturer Samsung -> muRata; Note 0201 X6T 6.3V, DECD reservoir (Table 82) -> 0201 X5R 10V, DECD reservoir (Table 82) Code re-verified 20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; Price@1k $0.0091 -> $0.0301
- C6: LCSC Part # C2827888 -> C76941; MPN CL03A225MQ3CSNC -> GRM033R71A103KA01D; Manufacturer Samsung -> muRata; Note 0201 X7R - Table 82 lists it, Figure 175's extraction does not place its node. Wired to DECD. CANNOT DETERMINE against the source. -> 0201 X7R - Table 82 lists it, Figure 175's extraction does not place its node. Wired to DECD. CANNOT DETERMINE against the source. Code re-verified 2026-09-05 (S1).; Price@1k $0.0091 -> $0.0301
- C7: LCSC Part # C2827888 -> C161479; MPN CL03A225MQ3CSNC -> GRM033R71A222KA01D; Manufacturer Samsung -> muRata; Note 0201 X7R - same, CANNOT DETERMINE -> 0201 X7R - same, CANNOT DETERMINE Code re-verified 2026-09-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; Price@1k $0.0091 -> $0.0301
- C8: LCSC Part # C2827888 -> C335106; MPN CL03A225MQ3CSNC -> GRM033R61A225KE47D; Manufacturer Samsung -> muRata; Note 0201 X6T, on the DECA=DECRF node -> 0201 X5R 10V, on the DECA=DECRF node. Code re-verified 2026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; Price@1k $0.0091 -> $0.0301
- L1: LCSC Part # C1046 -> C76799; Note 0603 multilayer, >=120 mA Isat, DCC->DECD. 0603 is 0.9 mm t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 -> 0603 multilayer, >=120 mA Isat, DCC->DECD. Code re-verified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; Price@1k $0.0180 -> $0.0301
- L10: LCSC Part # C25076 -> C473473; MPN 0201WMJ0000TEE -> 0201WMF0000TEE; Note PI SERIES, fitted as a 0 ohm jumper so the board works untuned. Replaced by an inductor if ce-rf's S11 asks for one. -> PI SERIES, fitted as a 0 ohm jumper so the board works untuned. Replaced by an inductor if ce-rf's S11 asks for one. Code re-verified 2026-09-05: C25076 is 100 R 0402 (S1).; Price@1k $0.0012 -> $0.0010
- L2: LCSC Part # C1046539 -> C7216765; Note 0201 LQP03HQ2N7B02, Nordic ref -> 0201 LQP03HQ2N7B02, Nordic ref Code re-verified 2026-09-05 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; Price@1k $0.0304 -> $0.0168
- L3: LCSC Part # C1046539 -> C3911055; MPN LQP03HQ2N7B02D -> LQP03HQ3N5B02D; Note 0201 LQP03HQ3N5B02, Nordic ref -> 0201 LQP03HQ3N5B02, Nordic ref Code re-verified 2026-09-05 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; Price@1k $0.0304 -> $0.0168
- L4: LCSC Part # C1046539 -> C3911055; MPN LQP03HQ2N7B02D -> LQP03HQ3N5B02D; Note 0201, = L3, Nordic ref -> 0201, = L3, Nordic ref Code re-verified 2026-09-05 (S1).; Price@1k $0.0304 -> $0.0168
- R1: LCSC Part # C25765 -> C778408; Note sense divider, high leg -> sense divider, high leg. Code re-verified 2026-09-05: C2576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; Price@1k $0.0012 -> $0.0015
- R10, R6, R7, R8: LCSC Part # C25744 -> C473048; Price@1k $0.0012 -> $0.0010
- R2: LCSC Part # C25765 -> C778408; Price@1k $0.0012 -> $0.0015
- R5: LCSC Part # C25744 -> C473048; Note CS strapped HIGH = I2C mode (DS11811 §5). Through a resistor, not a via, so SPI can be selected on a bring-up board by moving it. -> CS strapped HIGH = I2C mode (DS11811 §5). Through a resistor, not a via, so SPI can be selected on a bring-up board by moving it. Code re-verified 2026-09-05: C25744 is 0402 under an 0201 land (S1).; Price@1k $0.0012 -> $0.0010
- R9: LCSC Part # C25076 -> C270366
- X1: LCSC Part # C32346 -> C95361; MPN FC-135 32.768kHz -> Q13FC13500049; Note Epson 32.768 kHz. CHANGED from X321532768KGD2SI (C620155) o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 -> Epson FC-135 32.768 kHz, CL = 6 pF. CHANGED from C32346 (Q1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; Price@1k $0.1375 -> TBC; Stock 444,985 -> 134,310
- X2: MPN NX2016SA-32MHZ -> NX2016SA-32MHZ-STD-CZS-5; Note CL 8 pF, +/-10 ppm, 2.0x1.6x0.5 mm. Nordic's BOM says a 2-pad 2016 and KiCad ships no 2-pin 2016 land pattern, so the 4-pad symbol is used and the can is grounded - better RF practice anyway. Recorded as a substitution. -> CL 8 pF, +/-10 ppm, 2.0x1.6x0.5 mm. Nordic's BOM says a 2-pad 2016 and KiCad ships no 2-pin 2016 land pattern, so the 4-pad symbol is used and the can is grounded - better RF practice anyway. Recorded as a substitution. MPN completed to the orderable suffix 2026-09-05.
