File: out/verify/halo_rev_a.kicad_pcb (KiCad board)
At the start: 4 copper layers, 25.6 x 26 mm, 62 parts, among them J1 TC2030, J2 UWB stub, U1 nRF54L10-QFAA-R7, U2 LIS2DW12TR, X1 32.768kHz, X2 32MHz

Commit message: checkpoint: board and verification work in flight when the machine crashed 03:32
Committed as-is so it survives, NOT as a result. Measured right now: board DRC
12 violations; the drill blocker looks closed — PTH.drl carries 50 holes against
49 vias declared in the board, which needs confirming rather than assuming (a
PTH file also carries through-hole pads).

B1 built a verification suite in out/verify/: bom-identity, cpl-rotations and
lcsc-netlist PASS; dfm-jlc-4layer, fabset and convergence-integrity FAIL.

Co-Authored-By: Claude Opus 5 (1M context) <noreply@anthropic.com>
Claude-Session: https://claude.ai/code/session_01DLBM9xzZTSLgvB55tmrcPa
Parts:
- AE2: footprint HALO_NFC_TIE_2 -> NetTie-2_SMD_Pad0.5mm
- turned AE2 to -129.117 degrees
Routing:
- net GND: track 8.79 -> 9.67 mm
- net VDD: track 7.34 -> 7.92 mm, vias 9 -> 10

Commit message: convergence: a source that resolves to nothing was grading better than a literal
Three fixes to the integrity check and the table it grades, each found by
running the check rather than reading it.

1. `elif src:` PASSED ON THE STRING IN THE `from` FIELD. G6 high_weight_measured
exists to catch a weight-10 claim whose current value is typed into the spec.
It compared `from` to the word "literal" and passed everything else — so a row
naming a source that produced NO VALUE scored better than one that honestly
typed the number in. Measured: two antenna rows (radiation efficiency, realized
gain) were reading PASS on G6 with `current: null`, because their ce-rf case had
FAILED and rf() correctly refused its numbers. They are CANNOT DETERMINE now.

2. THREE BOARD ROWS WERE LITERALS WHOSE VALUES WERE ALREADY ON DISK. Layer
count, PCB outline diameter and PCB thickness are all in
out/verify/dfm-jlc-4layer.json's board_facts, measured by ce-fab's own parser
off the .kicad_pcb. New source kind `from: "file"` (path + dotted pointer +
optional max/min reduce) reads them, and returns None with a stated reason when
the file or the key is missing. New assertion G8 source_file_resolves fails a
row whose named file or key does not exist — without it, `file` would have been
a fourth way to score a PASS for naming something.

3. "DELIBERATE DIVERGENCE" WAS A ROW THAT COULD NOT BE WRONG. PCB thickness had
no numeric target, only the text "0.30 mm — deliberately NOT matched", so the
state machine answered OPEN for the right value and for a deliberately wrong one
— G1 said so and it was right. The row now carries Apple's real 0.30 mm as its
target and a `divergence` block naming D17 and the 0.60 mm we committed to: land
on 0.60 and the row reads DIVERGENT, land anywhere else and it reads OPEN like
any other row. New assertion G9 divergence_is_earned refuses a divergence with
no decision behind it, and refuses one whose own value sits INSIDE the target's
tolerance — that is a MATCH relabel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
Parts:
- AE2: footprint NetTie-2_SMD_Pad0.5mm -> HALO_NFC_TIE_2
- turned AE2 to 128.883 degrees
Routing:
- net GND: track 9.67 -> 8.79 mm
- net VDD: track 7.92 -> 7.34 mm, vias 10 -> 9
