File: electronics/halo_replica/pcb/out/halo_replica.kicad_pcb (KiCad board)
At the start: 4 copper layers, 24.7 x 24.7 mm, 108 parts

Commit message: E07 synthesis: three kinds of adjacent, and the pipeline exit code as a sixth
Refinement from the comparison lane: the five cases differ in WHAT the adjacent
property was - three adjacent STATISTICS (increment permutation, off-peak noise,
area alone), one adjacent COORDINATE (between-in-x), one adjacent PATH (a guard
resolving against the search root). The path case is the one people least expect
because it is not a modelling error at all - a plumbing error wearing a control's
clothes, which no amount of thinking about the physics would have found.

Plus a sixth of the same shape from the same day: reading 'cmd | tail's exit
status instead of the command's. PIPESTATUS[0] gives the real one. The exit code
you read was adjacent to the exit code you wanted.

Co-Authored-By: Claude Opus 5 (1M context) <noreply@anthropic.com>
Claude-Session: https://claude.ai/code/session_01JRY3feHovaK2VS3mL7infx
Parts:
- B002: value MEASURED METAL 2.05x2.54 mm conf=high -> MEASURED METAL 2.05x2.54 mm at 99.5727 deg conf=high
- B003: value MEASURED METAL 2.25x2.69 mm conf=high -> MEASURED METAL 2.25x2.69 mm at 124.8366 deg conf=high
- B004: value MEASURED METAL 0.98x5.4 mm conf=high -> MEASURED METAL 0.98x5.4 mm at 152.0923 deg conf=high
- B005: value MEASURED METAL 1.15x3.88 mm conf=high -> MEASURED METAL 1.15x3.88 mm at 125.1839 deg conf=high
- B006: value MEASURED METAL 0.79x4.49 mm conf=high -> MEASURED METAL 0.79x4.49 mm at 99.8955 deg conf=high
- B007: value MEASURED METAL 0.78x4.47 mm conf=high -> MEASURED METAL 0.78x4.47 mm at 28.9318 deg conf=high
- B008: value MEASURED METAL 1.4x1.71 mm conf=high -> MEASURED METAL 1.4x1.71 mm at 92.4532 deg conf=high
- B009: value MEASURED METAL 1.31x1.64 mm conf=high -> MEASURED METAL 1.31x1.64 mm at 176.7348 deg conf=high
- B010: value MEASURED METAL 1.72x2.32 mm conf=high -> MEASURED METAL 1.72x2.32 mm at 101.4441 deg conf=high
- B011: value MEASURED METAL 1.25x1.26 mm conf=high -> MEASURED METAL 1.25x1.26 mm at 49.9126 deg conf=high
- B013: value MEASURED METAL 1.21x2.87 mm conf=high -> MEASURED METAL 1.21x2.87 mm at 13.0051 deg conf=high
- B014: value MEASURED METAL 0.69x1.4 mm conf=high -> MEASURED METAL 0.69x1.4 mm at 63.4106 deg conf=high
- B015: value MEASURED METAL 0.81x1.95 mm conf=high -> MEASURED METAL 0.81x1.95 mm at 170.8109 deg conf=high
- B017: value MEASURED METAL 0.62x1.4 mm conf=high -> MEASURED METAL 0.62x1.4 mm at 71.0021 deg conf=high
- B019: value MEASURED METAL 0.55x1.34 mm conf=high -> MEASURED METAL 0.55x1.34 mm at 64.2329 deg conf=high
- B020: value MEASURED METAL 0.68x1.51 mm conf=high -> MEASURED METAL 0.68x1.51 mm at 5.7833 deg conf=high
- B023: value MEASURED METAL 0.74x1.59 mm conf=high -> MEASURED METAL 0.74x1.59 mm at 139.6705 deg conf=high
- B024: value MEASURED METAL 0.75x1.52 mm conf=high -> MEASURED METAL 0.75x1.52 mm at 131.5344 deg conf=high
- B025: value MEASURED METAL 0.8x1.57 mm conf=high -> MEASURED METAL 0.8x1.57 mm at 146.5259 deg conf=high
- B026: value MEASURED METAL 0.8x1.62 mm conf=high -> MEASURED METAL 0.8x1.62 mm at 145.5884 deg conf=high
- B028: value MEASURED METAL 0.6x0.9 mm conf=high -> MEASURED METAL 0.6x0.9 mm at 61.1923 deg conf=high
- B029: value MEASURED METAL 0.56x0.71 mm conf=high -> MEASURED METAL 0.56x0.71 mm at 126.6338 deg conf=high
- B030: value MEASURED METAL 0.55x0.73 mm conf=high -> MEASURED METAL 0.55x0.73 mm at 127.0454 deg conf=high
- B034: value MEASURED METAL 0.51x0.7 mm conf=high -> MEASURED METAL 0.51x0.7 mm at 114.2637 deg conf=high
- B035: value MEASURED METAL 0.54x0.94 mm conf=high -> MEASURED METAL 0.54x0.94 mm at 54.6639 deg conf=high
- B046: value MEASURED METAL 0.7x1.49 mm conf=high -> MEASURED METAL 0.7x1.49 mm at 157.835 deg conf=high
- B064: value MEASURED METAL 1.02x3.21 mm conf=high -> MEASURED METAL 1.02x3.21 mm at 130.3 deg conf=high
- D000: value MEASURED METAL 3.03x3.28 mm conf=high -> U1 nRF52832-CIAA WLCSP-50 - 56 LANDS DRAWN, 6 UNKNOWN; A1 CORNER CANNOT DETERMINE; body measured 3.28x3.03 mm here; footprint REPL_METAL_3.03x3.28 -> REPL_WLCSP_8x7_P0.4_GRID56
- D002: value MEASURED METAL 0.91x1.18 mm conf=high -> MEASURED METAL 0.91x1.18 mm at 154.8 deg conf=high
- D003: value MEASURED METAL 0.94x0.95 mm conf=high -> MEASURED METAL 0.94x0.95 mm at 3.7 deg conf=high
- D004: value MEASURED METAL 0.51x1.53 mm conf=high -> MEASURED METAL 0.51x1.53 mm at 85.7 deg conf=high
- turned B002 to -9.57273 degrees
- turned B003 to -34.8366 degrees
- turned B004 to -62.0923 degrees
- turned B005 to -35.1839 degrees
- turned B006 to -9.8955 degrees
- turned B007 to 61.0682 degrees
- turned B008 to -2.45315 degrees
- turned B009 to -86.7348 degrees
- turned B010 to -11.4441 degrees
- turned B011 to 40.0874 degrees
- turned B013 to 76.9949 degrees
- turned B014 to 26.5894 degrees
- turned B015 to -80.8109 degrees
- turned B017 to 18.9979 degrees
- turned B019 to 25.7671 degrees
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