File: electronics/halo_replica/pcb/out/halo_replica.kicad_pcb (KiCad board)
At the start: 4 copper layers, 24.7 x 24.7 mm, 150 parts

Commit message: L12: the back face, the mask colour, and two checks that caught themselves
BACK FACE — Apple's second populated side, drawn for the first time. 41
measured round gold pads (population median 0.5985 mm, IQR 0.0340) and 3
battery-contact POSITIONS, from lane L9's HANDOFF-positions-back.json.

THE HANDEDNESS IS MEASURED, NOT ASSUMED, and it is the thing that would
have been silently wrong. Both handoffs say "+x right, +y DOWN" IN THEIR OWN
PHOTOGRAPH; a board has one frame, so one of them is mirrored and neither
file says which. Get it wrong and all 43 pads land at (-x, y): the board
still builds, DRC still passes, the render still looks like a board.
tools/f_backface_handedness.py settles it from the outline angles of the
same physical board in FCC photo 6 and photo 7 — a MIRROR reproduces both
angles to 1.00 deg while a ROTATION's implied k disagrees between them by
6.00 deg. Cross-check: the O'Flynn frame's largest chord normal is 0.98 deg
from photo 6's, so the homography preserves bearing. to_board_back() REFUSES
TO RUN if that verdict is not on disk.

THE FIRST NEGATIVE CONTROL FOR IT WAS VOID AND WAS WATCHED BEING VOID. It
swapped the two files' angles — but a reflection is its own inverse, so the
tool returned MIRROR both ways: an assertion agreeing with itself. Replaced
by one that SYNTHESISES a rotated back face, and MIRROR is correctly refused
at 12, 40 and 90 deg.

SOLDERMASK — black, from stackup.json's replica_as_drawn, a CHOICE inside
the measured bound "dark and neutral" (V 65-128, R/G/B within ~10 counts).
Apple's colour stays CANNOT DETERMINE; the refusal to call it purple travels
with it. THE SAME MISTAKE HAPPENED HERE AND WAS CAUGHT THE SAME WAY:
board._rules["soldermask_colour"] is a SILENT NO-OP, so the stackup block is
written into the s-expression and the file reloaded with pcbnew to prove it.
That check passed and THE BOARD STILL RENDERED GREEN, because kicad-cli
ignores the stackup without --use-board-stackup-colors. So the check moved
to the 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
Parts:
- added SILK3: silkscreen legend, tangential, REPL_SILK_THICKNESS, F.Cu at (22.7, 5.20)
- SILK1: value silkscreen legend, tangential -> silkscreen legend, radial
- SILK2: value silkscreen legend, radial -> silkscreen legend, tangential
- moved SILK2 15.8 mm to (22.5, 9.15), turned to -68 degrees
- moved SILK1 15.6 mm to (12.0, 21.4), turned to -108 degrees
