File: electronics/halo_replica/out/schematic/halo_replica.kicad_sch (KiCad schematic)
At the start: 68 parts, among them J1 COAXIAL RF RECEPTACLE, U.FL/I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, U1 nRF52832-CIAA (WLCSP-50) - DR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, U2 APPLE U1 UWB SiP - DNP / UNPO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, U3 GD25LQ32C 32Mb 1.8V SPI NOR (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, U4 3-AXIS ACCELEROMETER - PART C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, U5 MAX98357A-CLASS CLASS-D AMP (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, U6 TPS62746-CLASS BUCK 3V->1V8 (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, U7 TLV9001-CLASS OP-AMP - ROLE I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, U8 FPF2487-CLASS LOAD SWITCH (LO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, U9 CANNOT DETERMINE - marking 1A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, X1 32 MHz? marking T320 / RBEV -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, X2 32.768 kHz? marking A048L - P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

Commit message: L8: J1 measured - it is NOT a U.FL, and the exclusion is a factor of 1.4-1.7
THE RESULT. J1's metal shell measures 1.860 x 1.707 mm (b_pkgsize --fill-holes,
pad sweep 0/20/40/60 px STABLE at 0.08% / 0.39%). Against Hirose's own U.FL-R-SMT-1
outline - 2.6 mm square body, 3.0 x 3.1 mm overall, Ø2.0 mm shell, read out of the
Hirose U.FL catalogue PDF - that is -28%/-34% on the square and -38%/-45% on the
overall. Nothing in the +/-1% scale band or the +/-4% segmentation band spans that,
and the measurement is already an over-estimate (b_pkgsize reads 3.5-3.9% high and
the extent INCLUDES the four solder tabs). U.FL IS EXCLUDED.

What it IS: 1.860 x 1.707 mm sits 7.0% and 3.0% inside the MHF4 receptacle's
2.00 x 1.76 mm housing - read out of I-PEX's own 2D drawing 20449C15 rev 15 - which
is the right sign and roughly the right size, because that housing is black LCP and
extends past the bright metal that was segmented. W.FL / Murata HSC sit within a few
percent of MHF4 and CANNOT be separated from it here, and that is said rather than
guessed.

Both published figures were FETCHED AND READ, not recalled. The BOM had carried
"U.FL is 2.6 mm, MHF4 is 2.0 mm" with no source; the whole exclusion rests on them.
Wikipedia's comparison table is cited as SECONDARY and used only for W.FL, because
its MHF4 row (1.7 x 1.7) disagrees with I-PEX's own drawing (1.76 x 1.68).

Corroboration reported WITH its weakness: boardmetro circles over 1.2-2.6 mm found
exactly one maximum above its own null bar - d = 1.700 mm, closure 1.22 against a bar
of 0.69 - but noncircularity 0.718 and inlier fraction 0.376, because the four tabs
break the ring. It corroborates the barrel's scale and is not a second measurement.

TOOLING. b_pkgsize gains --fill-holes, and this part is why: a connector is a RING,
it fills 0.469 of its own bounding rectangle, under the 0.60 rectangularity floor,
and the tool REFUSED one of the most unambiguous objects on the board. The floor is
right - it is what rejects thre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
Parts:
- ANT1: value BLE 2.4 GHz INVERTED-F, PRINTED ON THE CARRIER -> BLE 2.4GHz INVERTED-F (on carrier)
- ANT2: value NFC COIL - WOUND MAGNET WIRE, >=9 TURNS (LOWER BOUND) -> NFC COIL - WOUND WIRE, >=9 TURNS
- ANT3: value UWB PATCH 6.5/8 GHz, PRINTED ON THE CARRIER -> UWB PATCH 6.5/8GHz (on carrier)
- BT1: value 3 SPRUNG CONTACTS (1 neg dome, 2 pos tabs) -> 3 SPRUNG CONTACTS (1 neg, 2 pos)
- C1, C2, C3, C4, C5: value 100uF (marking J107S) - TECHNOLOGY CANNOT DETERMINE -> 100uF? mark J107S - CANNOT DETERMINE
- C10, C11, C12, C13: value DECOUPLING - VALUE CANNOT DETERMINE -> DECOUPLING - CANNOT DETERMINE
- C14, C15, C16, C17: value VALUE CANNOT DETERMINE -> CANNOT DETERMINE
- C18, C19, C20, C21: value LOAD CAP - VALUE CANNOT DETERMINE -> LOAD CAP - CANNOT DETERMINE
- C6, C7: value NFC TUNING - VALUE CANNOT DETERMINE -> NFC TUNING - CANNOT DETERMINE
- C8, C9: value PI SHUNT - VALUE CANNOT DETERMINE -> PI SHUNT - CANNOT DETERMINE
- J1: value COAXIAL RF RECEPTACLE, U.FL/IPEX MHF-CLASS BY CONSTRUCTION - EXACT PART CANNOT DETERMINE -> COAX RF RECEPTACLE - PART CANNOT DETERMINE; BOM confidence HIGH that a coaxial RF receptacle is fitted at this location on this unit. -> HIGH that a coaxial RF receptacle is fitted at this location on this unit. HIGH that it is NOT a U.FL — the size difference is far outside any error here. CANNOT DETERMINE which of; BOM part CANNOT DETERMINE — a U.FL / IPEX MHF-class receptacle by co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 -> CANNOT DETERMINE for the part number. MEASURED to be of the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
- L1: value WIREWOUND CHIP INDUCTOR - VALUE CANNOT DETERMINE -> WIREWOUND - CANNOT DETERMINE
- L2: value DC/DC INDUCTOR - VALUE CANNOT DETERMINE -> DC/DC L - CANNOT DETERMINE
- L3: value PI SERIES - VALUE CANNOT DETERMINE -> PI SERIES - CANNOT DETERMINE
- LS1: value VOICE COIL - WOUND MAGNET WIRE, GLUED TO THE DOME -> VOICE COIL - WOUND MAGNET WIRE
- R1: value SENSE TOP, P+_POWER - VALUE CANNOT DETERMINE (~50 nA implies megohms) -> SNS TOP P+_PWR - CANNOT DETERMINE
- R10: value SENSE DIVIDER BOT - VALUE CANNOT DETERMINE -> SENSE DIV BOT - CANNOT DETERMINE
- R2: value SENSE BOTTOM, P+_POWER - VALUE CANNOT DETERMINE (~50 nA implies megohms) -> SNS BOT P+_PWR - CANNOT DETERMINE
- R3: value SENSE TOP, P+_SENSE - VALUE CANNOT DETERMINE (~50 nA implies megohms) -> SNS TOP P+_SNS - CANNOT DETERMINE
- R4: value SENSE BOTTOM, P+_SENSE - VALUE CANNOT DETERMINE (~50 nA implies megohms) -> SNS BOT P+_SNS - CANNOT DETERMINE
- R5, R6: value I2C PULL-UP - VALUE CANNOT DETERMINE -> I2C PULL-UP - CANNOT DETERMINE
- R8: value GAIN STRAP - VALUE CANNOT DETERMINE -> GAIN STRAP - CANNOT DETERMINE
- R9: value SENSE DIVIDER TOP - VALUE CANNOT DETERMINE -> SENSE DIV TOP - CANNOT DETERMINE
- TP28: value nRF CORE RAIL (DEC1) - THE GLITCH PAD -> nRF CORE RAIL - THE GLITCH PAD
- U1: value nRF52832-CIAA (WLCSP-50) - DRAWN AS QFAA/QFN-48 -> nRF52832-CIAA WLCSP-50 (drawn QFN-48)
- U2: value APPLE U1 UWB SiP - DNP / UNPOPULATED - NEVER SOLD TO ANYONE -> APPLE U1 UWB SiP - DNP, NEVER SOLD
- U3: value GD25LQ32C 32Mb 1.8V SPI NOR (WLCSP-10) - DRAWN AS WSON-8 -> GD25LQ32C 32Mb 1.8V NOR (WLCSP-10)
- U4: value 3-AXIS ACCELEROMETER - PART CANNOT DETERMINE (BMA280 is a teardown ASSERTION, not a marking) -> 3-AXIS ACCEL - PART CANNOT DETERMINE
- U5: value MAX98357A-CLASS CLASS-D AMP (LOW confidence; iFixit wrote MAX98357B) -> MAX98357A-CLASS AMP (LOW conf)
- U6: value TPS62746-CLASS BUCK 3V->1V8 (part MEDIUM, package CANNOT DETERMINE) -> TPS62746-CLASS BUCK 3V->1V8
- U7: value TLV9001-CLASS OP-AMP - ROLE INFERRED, LOW confidence -> TLV9001-CLASS OP-AMP - ROLE INFERRED
- U8: value FPF2487-CLASS LOAD SWITCH (LOW confidence, SILICON CITED, single-source) -> FPF2487-CLASS LOAD SWITCH (LOW conf)
- U9: value CANNOT DETERMINE - marking 1A8 / 1950; even 'regulator' is inferred -> CANNOT DETERMINE - mark 1A8/1950
- X1: value 32 MHz? marking T320 / RBEV - PART AND LOAD CAP CANNOT DETERMINE -> 32 MHz? mark T320/RBEV - CANNOT DETERMINE
- X2: value 32.768 kHz? marking A048L - PART AND LOAD CAP CANNOT DETERMINE -> 32.768 kHz? mark A048L - CANNOT DETERMINE
Other:
- title: halo REPLICA - Apple AirTag A2187 reconstructed. NO COPPER WAS TRACED: every net is INFERRED or CHOSEN unless marked MEASURED. -> halo REPLICA - Apple AirTag A2187, reconstructed
- moved on the sheet: ANT1, ANT2, ANT3, C10, C11, C12, C13, C14, C15, C16, C17, C18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

Commit message: L11: I never LOOKED at the drawing, and three things were wrong on it
Every number on this sheet was green and every check passed. Then I rendered
it and looked, which is a standing rule I had not obeyed on my own
deliverable.

WHAT THE PICTURE SHOWED, none of which any check could see:

1. THE VALUE FIELDS WERE PARAGRAPHS. 29 of 68 ran over 40 characters, up to
   92, and each is drawn beside its symbol — they landed on their neighbours.
   Now none exceeds 45; the prose was already in each part's Note field,
   which is where a reader who wants it looks.
2. THE SHEET NOTES WERE DRAWN OFF THE PAGE. 16 paragraph-length notes into
   about 14 lines of room, the rest printed past the bottom edge over the
   frame and over each other. Fixed in ce-pcb (208016f9, a7eb2c4b) and cut to
   SIX here — a schematic was never the place to keep all of it, and the rest
   is in this file's docstring and NETS.md.
3. THE TITLE was 126 characters into a fixed-width block, so it was truncated
   mid-sentence. Short now; the claim it carried is a sheet note.

And looking properly mattered twice over: at page scale the note block LOOKED
like it had overlapping lines, and the measurement said it fitted with 34 mm
to spare. At real zoom the notes were clean — but the rail strip's GND label
was printing on top of the first note line, which page scale had hidden. Two
opposite errors of eye in one image; only the zoom settled either.

J1 IS NOT A U.FL AND THIS SHEET CALLED IT ONE TWICE. The metrology lane
measured the shell at 1.860 x 1.707 mm; a Hirose U.FL-R-SMT-1 is a 2.6 mm
square body, 3.0 x 3.1 mm overall — -28%/-34% and -38%/-45%, and the
measurement is already an over-estimate because it includes the four
protruding tabs. No error band here spans a 28-45% gap. It is MHF4-class;
W.FL and Murata HSC are within a few percent and cannot be separated.
THE U.FL FOOTPRINT WENT WITH THE WORD: a land pattern from the wrong
connector family is a board that cannot be assembled, and it had been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
Parts:
- J1: value COAX RF RECEPTACLE - PART CANNOT DETERMINE -> COAX RF RECEPTACLE, MHF4-CLASS - PART CANNOT DETERMINE; footprint Connector_Coaxial:U.FL_Hirose_U.FL-R-SMT-1_Vertical -> (none); Excluded by measurement (none) -> U.FL (2.6 mm square body, 3.0 x 3.1 mm overall); FP-basis SUBSTITUTION -> PLACEHOLDER-L12; Measured (none) -> 1.860 x 1.707 mm shell incl. tabs; Note THIS PART REFUTES 'CONNECTORS: NONE ANYWHERE', which REFERENCE-TEARDOWN 2.5 states and SPEC.md repeats. A circular RF receptacle - metal outer shell, four solder tabs, dark dielectric annulus, gold centre contact - is unambiguous at 5x on the component face. HIGH confidence that it is fitted on this unit. WHICH receptacle (U.FL vs one of the MHF variants) is a SUBSTITUTION; the Hirose land pattern is the family's common one. -> THIS PART REFUTES 'CONNECTORS: NONE ANYWHERE', which REFERENCE-TEARDOWN 2.5 states and SPEC.md repeats. A circular RF receptacle - metal outer shell, four solder tabs, dark dielectric annulus, gold centre contact - is unambiguous at 5x on the component face. MEASURED 1.860 x 1.707 mm (shell including tabs), which EXCLUDES U.FL by 28-45% against Hirose's own catalogue and sits 7.0% / 3.0% inside an MHF4 receptacle's 2.00 x 1.76 mm housing - the right sign, because that housing is black LCP extending past the bright metal segmented. W.FL and Murata HSC are within a few percent of MHF4 and CANNOT BE SEPARATED from it here. KiCad ships no MHF4 or W.FL land pattern, so this part has NO FOOTPRINT rather than the wrong one.
Other:
- note added: "D3 IS AN ADDITION, NOT AN OBSERVATION (DECISIONS.md D24). nRF52832 spec 42.10: a strong NFC field pushes current BACKWARDS into the supply through parasitic diodes, and a CR2032 does not tolerate return current. COST: a Schottky drops a few hundred mV against a cell already tracked to 68 mV of end-of-life droop; an ideal-diode controller drops millivolts and costs money. NO PHOTOGRAPH HERE SHOWS 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"
- note added: "FOUR PARTS THAT ARE ON THE REAL BOARD AND NOT ON THIS SHEET, because placing a part asserts what it is: D1/D2 (marking K11), CT1 ('6X A75', and 'blue' is a colour, not a technology), UNK-A and UNK-B. TP1/TP38 are absent too - REFERENCE-TEARDOWN and Apple's own FCC arrow disagree about which coil that annulus is. EVERY PASSIVE VALUE HERE IS CANNOT DETERMINE and stays that way: a 100 nF and a 1 uF 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"
- note added: "J1 REFUTES 'CONNECTORS: NONE ANYWHERE' - REFERENCE-TEARDOWN 2.5 says it and SPEC.md repeats it. IT IS ALSO NOT A U.FL, which this sheet called it twice: the shell MEASURES 1.860 x 1.707 mm against a U.FL's 2.6 mm square body, -28% to -45%, a gap no error band here spans. MHF4-class; W.FL and Murata HSC are within a few percent and cannot be separated. KiCad ships no such land pattern, so J1 has N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"
- note added: "THE PACKAGES ARE NOT APPLE'S PACKAGES. U1 is an nRF52832-CIAA, WLCSP-50, drawn with the QFN-48 (QFAA) symbol of the SAME DIE because no COMPLETE ball map is sourced here - O'Flynn's table gives TEN of the fifty (D3 E2 F1 F4 G1 G3 H1 H2 H3 H4). U3 is a WLCSP-10 drawn as WSON-8, U5 a WLCSP drawn as TQFP-16. THE NETLIST IS RIGHT BY SIGNAL NAME AND THE PIN NUMBERS ARE NOT APPLE'S. Every part carries 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"
- note added: "U2 IS APPLE'S 'U1' UWB SiP AND IT IS DNP / UNPOPULATED. Apple does not sell it to anyone, at any price, with any lead time - not a sourcing problem but a does-not-exist-for-us one, which is why Precision Finding is a GAP and not a to-do. ITS PIN NUMBERS HERE ARE INVENTED: no pinout for that module has ever been published, so its land pattern does not exist and NOTHING MAY BE FABRICATED FROM IT. (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"
- note added: "U4 AND U9 ARE CANNOT DETERMINE. Two visually identical metal-lid parts are on the board and neither is confidently the accelerometer; 'BMA280' is a teardown assertion this project failed to corroborate. U9, marked '1A8 / 1950', is unidentified DOWN TO ITS FUNCTION, so its output is wired to nothing rather than to a plausible load."
- note added: "halo REPLICA - Apple AirTag A2187 (FCC ID BCGA2187), reconstructed. NOBODY HAS TRACED APPLE'S COPPER: 13 of 52 nets are MEASURED and each names a file and a string checked at build time; the other 39 are 21 INFERRED and 18 CHOSEN. NEVER CITE A CHOSEN NET AS A FINDING ABOUT APPLE. Full table, with what drives each net and what it feeds: schematic/NETS.md."
- note removed: "A CONTRADICTION INSIDE O'FLYNN'S OWN TABLE, CARRIED NOT RESOLVED: row 8 reads 'nRF ball E2 (P0.16)' and row 19 reads 'nRF ball H3 (P0.16)'. Two different balls with one GPIO number; one is a transcription error. This sheet takes row 19 because the SPI block's four balls H3/H4/G3/F4 are a coherent group, and TP8 IS DELIBERATELY ABSENT rather than drawn on a guess."
- note removed: "D3 IS AN ADDITION, NOT AN OBSERVATION (DECISIONS.md D24). nRF52832 product spec 42.10: a strong NFC field can push current BACKWARDS into the supply through parasitic diodes and ESD structures, and a CR2032 does not tolerate return current. A phone on the tag is a strong field by design. COST: a Schottky drops a few hundred mV against a cell already tracked to 68 mV of end-of-life droop; an ideal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"
- note removed: "EVERY CAPACITOR AND RESISTOR VALUE ON THIS SHEET IS CANNOT DETERMINE, and that is not laziness. bom.json: 'This is not a gap that any photograph can close: a 100 nF and a 1 uF 0402 are visually identical.' A missing value stays missing. THIS BOARD IS NOT BUILDABLE AS DRAWN and saying so is the point."
- note removed: "FOUR NETS ON THIS SHEET WERE WRONG UNTIL A CHECK FORCED SOMEBODY TO OPEN THE FILE THEY ALREADY CITED. The flash bus was drawn on P0.12/P0.13/P0.14 as a free CHOICE. O'Flynn's test-point table gives it by pad, by nRF BALL and by GPIO: SCLK on P0.17 (ball G3), COPI on P0.16 (H3), CIPO on P0.15 (H4), CS on P0.11 (F4). Three of the four were wrong and the fourth was right by luck. The bus is MEASURED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"
- note removed: "FOUR PARTS THAT ARE ON THE REAL BOARD AND NOT ON THIS SHEET, because placing a part asserts what it is: D1/D2 (marking K11, a matched pair - part AND function CANNOT DETERMINE), CT1 (marking '6X A75', blue body - and 'blue' is a colour, not a technology), UNK-A (large matte-black rectangle, no marking at all) and UNK-B (pale ceramic square between U2 and J1 - if it is an RF switch then this sheet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"
- note removed: "J1 REFUTES 'CONNECTORS: NONE ANYWHERE', which REFERENCE-TEARDOWN 2.5 states and SPEC.md repeats. A U.FL/IPEX-class coaxial receptacle is unambiguous at 5x on the component face of O'Flynn's retail unit. Two documents in this repository are wrong and this schematic is where that became unavoidable."
- note removed: "NAME COLLISION: on this sheet U1 is the NORDIC MCU and U2 is the Apple UWB part, following bom.json and REFERENCE-TEARDOWN. The press calls the Apple part 'the U1'. Never write bare U1 about it."
- note removed: "TEN CIAA BALLS ARE SOURCED, AND FORTY ARE NOT. O'Flynn's table names nRF ball designators for D3, E2, F1, F4, G1, G3, H1, H2, H3 and H4. That is not a ball map and does not make one - the package here is still the QFN-48 substitution - but it is ten more than this sheet first claimed existed, and L12 should have them when it draws the WLCSP land."
- note removed: "THE PACKAGES ARE NOT APPLE'S PACKAGES. U1 is an nRF52832-CIAA, WLCSP-50, drawn with the QFN-48 (QFAA) symbol of the same die because no COMPLETE CIAA ball map is sourced here (ten balls are; forty are not). U3 is a WLCSP-10 drawn as WSON-8. U5 is a WLCSP drawn as TQFP-16. THE NETLIST IS RIGHT BY SIGNAL NAME AND THE PIN NUMBERS ARE NOT APPLE'S. Every part carries an FP-basis field; L12 owns the la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"
- note removed: "THE iFIXIT ARGUMENT IS NOW SETTLED BY MEASUREMENT, not by self-consistency. O'Flynn, verbatim: 'The nrf controls power to the SPI flash, so you need to override it by supplying 1.8V on test point 21', and 'most of time the flash is powered off and thus the pins are tri-stated'. The flash sits on a switched 1.8 V rail the MCU commands - which is what this sheet drew from the argument that a load s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"
- note removed: "THIS SHEET DEPARTS FROM iFIXIT ON ONE THING AND SAYS SO: iFixit has the load switch U8 gating 'U1 + flash' where U1 is the MCU. A load switch whose enable comes from the MCU it powers can never be turned on. Here U8 gates the FLASH and the UWB module and the MCU sits on the 1.8 V rail directly."
- note removed: "TP1 AND TP38 ARE DELIBERATELY ABSENT. The fine coil leads land there; REFERENCE-TEARDOWN 2.4 calls them the VOICE COIL's joints and Apple's own arrow in FCC photo 5 labels that annulus the NFC ANTENNA. Both cannot be true and this sheet does not pick a winner."
- note removed: "U2 IS APPLE'S 'U1' UWB SiP AND IT IS DNP / UNPOPULATED. Apple does not sell it to anyone, at any price, with any lead time. That is not a sourcing problem, it is a does-not-exist-for-us problem, and Precision Finding is therefore a GAP and not a to-do. Its pin NUMBERS on this sheet are invented: no pinout for this module has ever been published, so its land pattern does not exist and NOTHING MAY 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"
- note removed: "U4 IS CANNOT DETERMINE. Two visually identical metal-lid parts are on the board and neither is confidently the accelerometer; no marking is readable at any magnification available here. 'BMA280' is a teardown assertion this project failed to corroborate. The symbol is generic and the value field says so."
- note removed: "U9 IS CANNOT DETERMINE, INCLUDING ITS FUNCTION. Marking '1A8 / 1950'. Its output is deliberately wired to NOTHING, because the record does not say what it feeds and a wire to a plausible load would be this sheet inventing a circuit."
- note removed: "halo REPLICA - Apple AirTag A2187 (FCC ID BCGA2187), reconstructed. NOBODY HAS TRACED APPLE'S COPPER. Every net carries a basis - MEASURED, INFERRED or CHOSEN - and NETS.md beside this file lists all of them with the counts DERIVED, never typed. 13 of 52 nets are MEASURED, and every one of those names a FILE AND A STRING THAT MUST BE IN IT, checked at build time. The other 39 are inference and ch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"
- moved on the sheet: ANT1, ANT2, ANT3, C10, C11, C12, C13, C14, C15, C16, C17, C18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
