File: electronics/halo_replica/out/schematic-fab/halo_replica_fab.kicad_sch (KiCad schematic)
At the start: 45 parts, among them J1 VOICE COIL / SOUNDER, J2 NFC COIL 13.56MHz, J3 SWD (nRST SWDIO SWCLK GND VBA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, U1 nRF52832-QFAA-R, U2 MIC94090YC6 (0.5 uA, 1.5 A), U3 MX25R3235F 32Mb 1.65-3.6V, U4 SC7A20 3-axis, LGA-12, U5 MAX98357A class-D, TQFN-16, X1 32MHz 10ppm CL=8pF, X2 32.768kHz 20ppm CL=12.5pF

Commit message: L11 fab: the size difference is a FORK, not a compromise, and it says so on the drawing
Power decision confirmed by the orchestrator: run from the cell, no buck,
keep the MX25R3235F. Nothing changed for that — this commit is the one thing
in the reply that was mine to act on.

"THIS BOARD IS NOT THE SIZE OF AN AIRTAG" was in U1's Package-delta field.
That is not enough: it has to survive into every downstream artifact, and a
field on one part does not travel. It is now a sheet note, in the words that
make it a fork rather than a compromise:

  Apple's WLCSP-50 FITS the ~6 mm annular ring and CANNOT BE LANDED, because
  no complete ball map for it has ever been published. The QFN-48 is the
  same die, CAN be landed, and is 6x6 mm — which does not fit that ring.
  There is no arrangement that is both. This is the BUILDABLE branch; the
  dimensional branch is the metrology record in pcb/, where the 0.30 mm
  board and the wafer-scale packages live.

A person holding a board that works but is the wrong shape should not have to
work out why. U1's field carries the same words and tells the reader to carry
them downstream.

NOT_VERIFIED reordered so "NOBODY HAS BUILT ONE" is FIRST rather than last,
and says why it is first: a reader who stops after one line should stop after
that one. Everything else in that list is a paper claim underneath it.

Still A2, 45 parts, 37 nets, 149 pin connections, ERC PASS 0 errors /
4 warnings, no note refused. The fidelity sheet and its outputs are untouched
by this commit and still report 7/7 checks and 13 MEASURED / 21 INFERRED /
18 CHOSEN — verified, not assumed.

Co-Authored-By: Claude Opus 5 (1M context) <noreply@anthropic.com>
Claude-Session: https://claude.ai/code/session_013mLHcufSVJ7BYZ5QCYysr1
Parts:
- U1: Package delta QFN-48 6x6x0.9 mm vs Apple's WLCSP-50 3.0x3.2x0.5 mm - this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 -> QFN-48 6x6x0.9 mm vs Apple's WLCSP-50 3.0x3.2x0.5 mm. THIS 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
Other:
- note added: "THIS BOARD IS NOT THE SIZE OF AN AIRTAG, AND THAT IS A FORK RATHER THAN A COMPROMISE. Dimensional fidelity and buildability are in DIRECT CONFLICT here: Apple's WLCSP-50 fits the ~6 mm annular ring and CANNOT BE LANDED, because no complete ball map for it has ever been published. The QFN-48 is the same die, CAN be landed, and is 6x6 mm - which does not fit that ring. There is no arrangement that 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"
- moved on the sheet: AE1, C17, C18, C21, C22, C23, C24, C25, C3, C4, C5, C6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

Commit message: L11: the fab BOM exists, and resolving its order codes found a wrong one I had just written
"Files ready to send to JLCPCB" is gerbers + drill + CPL + A BILL OF
MATERIALS. L13 has the first three coming from the board; the BOM comes from
the schematic, so it is mine, and nothing in ce-pcb could produce one. That
capability is now upstream (ce-workshop 609a9fcb) and this is the halo half.

  out/schematic-fab/halo_replica_fab-bom.csv           25 lines, 44 parts
  out/schematic-fab/halo_replica_fab-bom-resolved.csv  + order codes and their sources

TWO DEFECTS ON MY OWN SHEET, BOTH FOUND BY THE NEW TOOLS RATHER THAN BY
READING:

1. bom_from_sch groups by value + footprint + MPN, and it split two 0402
   lines that looked identical. C10 is 1 uF and was carrying CL05B104KO5NNNC,
   a 100 nF part number; the 22 pF crystal loads were carrying an 8 pF one.
   One MPN pasted across a loop whose members have different values. The
   value was right, the footprint was right, only the order number was wrong,
   and nothing else on this sheet could have caught it. Fixed; the BOM went
   26 lines to 25 as C6 and C10 correctly merged.

2. x_lcsc_resolve's FIRST REAL RUN PRODUCED A WRONG ORDER CODE, from the tool
   whose own docstring says a wrong code is worse than no code. It matched
   the chip antenna's 2450AT18A100 against catalogue line 2450AT18A100E and
   returned C89334 — a different part number, matched because the shorter is
   a substring of the longer.

   IT WAS CAUGHT BY READING THE FIVE SOURCE LINES, NOT BY ANY CHECK. The
   self-test had a case for the other direction — a long schematic MPN
   against a short catalogue one — and passed, which is exactly how a
   one-directional test flatters. Matching is token-exact now (the characters
   either side must not be alphanumeric; \b cannot be used because real part
   numbers contain +, . and -), and BOTH directions are tested. Resolved
   lines went 5 to 4, which is the correct direction for a fix like this.

WHAT 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
Parts:
- C10: MPN CL05B104KO5NNNC -> CL05A105KA5NNNC
- C17, C18: MPN CL05C080CB5NNNC -> CL05C220JB5NNNC
Changed lines of the file:
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@@
 			)
 		)
-		(property "MPN" "CL05B104KO5NNNC"
+		(property "MPN" "CL05A105KA5NNNC"
 			(at 259.08 101.6 0)
 			(effects
@@
 			)
 		)
-		(property "MPN" "CL05C080CB5NNNC"
+		(property "MPN" "CL05C220JB5NNNC"
 			(at 351.79 39.37 0)
 			(effects
@@
 			)
 		)
-		(property "MPN" "CL05C080CB5NNNC"
+		(property "MPN" "CL05C220JB5NNNC"
 			(at 351.79 69.85 0)
 			(effects

Commit message: L11: the order-code resolver now checks the package too, and its parser was inventing absences
Working the 21 open MPNs. Four findings, and three of them are defects in my
own tooling caught before anything was published.

1. THE PARSER WAS MANUFACTURING MEASURED ABSENCES. The JLCPCB dump's
   manufacturer column is TRUNCATED to its width, so when a name fills it
   there is only ONE space before the package - "Johanson Dielectr 1206". My
   row regex demanded two, parsed ZERO rows for every such part, and those
   keywords then read as "searched and returned nothing".

   A PARSER THAT FAILS TO MATCH DOES NOT LOOK LIKE A PARSER THAT FAILED. It
   looks like an empty result, and here an empty result is a CLAIM - "the
   catalogue was queried and has nothing". Structured rows went 293 -> 383
   and searched-and-absent went 28 -> 13. FIFTEEN OF THE TWENTY-EIGHT
   ABSENCES I WAS ABOUT TO REPORT WERE MY OWN PARSER.

2. THE PACKAGE CHECK ANSWERED "I CANNOT TELL" TO EVERYTHING. `\b` does not
   match between "_" and a digit, so "C_0402_1005Metric" never matched and
   every imperial comparison returned CANNOT DETERMINE - including the one
   that should have said 0402-against-0603 is WRONG. A check that is
   cautious about everything is indistinguishable from a check that is
   working. Now (?<!\d)...(?!\d), and the 0402-vs-0603 case goes red.

3. A CODE IS NO LONGER ACCEPTED UNTIL ITS PACKAGE IS CHECKED against the land
   pattern on the sheet. Matching a part number is one claim; that the part
   arrives in the shape the board expects is another, and a 1206 part under
   an 0402 land is a wrong code arriving by a different door. package_agrees
   answers only "do these CONTRADICT" - PASS, FAIL, or CANNOT DETERMINE where
   a land pattern's name carries no size at all. It does not guess, because a
   guess here either invents agreement or invents an alarm.

4. THE ANTENNA MPN WAS THE ONE THAT COULD BE CLOSED, AND THE FIX WAS ON MY
   SIDE. There is no catalogue part ca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
Parts:
- AE1: MPN 2450AT18A100 -> 2450AT18A100E; Substitution basis Apple's 2.4 GHz antenna is an inverted-F PRINTED ON THE PLASTIC CARRIER, and its geometry is CANNOT DETERMINE. A chip antenna is CHOSEN because it works on a board of any outline and needs no carrier: this board is meant to be switched on, not to be the right shape. -> Apple's 2.4 GHz antenna is an inverted-F PRINTED ON THE PLASTIC CARRIER, and its geometry is CANNOT DETERMINE. A chip antenna is CHOSEN because it works on a board of any outline and needs no carrier: this board is meant to be switched on, not to be the right shape. THE MPN CARRIES ITS 'E': the catalogue has no part called 2450AT18A100, and x_lcsc_resolve matched that shorter string inside the longer 2450AT18A100E and returned a code for a part number this sheet did not name. Both ends were wrong and both are fixed - the matcher is token-exact, and this line now names what can actually be bought.
Changed lines of the file:
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@@
 			)
 		)
-		(property "MPN" "2450AT18A100"
+		(property "MPN" "2450AT18A100E"
 			(at 27.94 193.04 0)
 			(effects
@@
 			)
 		)
-		(property "Substitution basis" "Apple's 2.4 GHz antenna is an inverted-F PRINTED ON THE PLASTIC CARRIER, and its geometry is CANNOT DETERMINE. A chip antenna is CHOSEN because it works on a board of any outline and needs no carrier: this board is meant to be switched on, not to be the right shape."
+		(property "Substitution basis" "Apple's 2.4 GHz antenna is an inverted-F PRINTED ON THE PLASTIC CARRIER, and its geometry is CANNOT DETERMINE. A chip antenna is CHOSEN because it works on a board of any outline and needs no carrier: this board is meant to be switched on, not to be the right shape. THE MPN CARRIES ITS 'E': the catalogue has no part called 2450AT18A100, and x_lcsc_resolve matched that shorter string inside the longer 2450AT18A100E and returned a code for a part number this sheet did not name. Both ends were wrong and both are fixed - the matcher is token-exact, and this line now names what can actually be bought."
 			(at 27.94 193.04 0)
 			(effects

Commit message: L11: BT1's holder could not fit the board at any position; the only one that does is through-hole
Claimed from the board lane and verified before changing anything, because
accepting it would have saved me the work — which is precisely when to check.

I RE-MEASURED ALL TEN CR2032 HOLDERS in KiCad's Battery library from the
footprint files themselves, and reproduced the board lane's numbers to 0.01 mm
on every row:
  BatteryHolder_Keystone_1060_1x2032        32.90 x 21.40  diag 39.25   no
  BatteryHolder_MYOUNG_BS-07-A1BJ001_CR2032 27.41 x  6.30  diag 28.13   FITS
  Battery_Panasonic_CR2032-VS1N_Vertical    20.61 x  6.23  diag 21.53   FITS
  ... seven others, all diag > 30 mm
A rectangle fits inside a circle only if its DIAGONAL fits, so on a 30.0 mm
disc the Keystone 1060 was impossible AT ANY POSITION AND ANY ROTATION. A
placement solver cannot report that: it pushes the part around and converges.

WHAT IT LOOKED LIKE INSTEAD, and this is the part worth keeping: the 1060's
courtyard is WIDER THAN THE WHOLE BOARD, so every through-hole pad on the disc
fell inside it by construction and KiCad reported nine `pth_inside_courtyard`
violations naming J3's pads. A PART-CHOICE PROBLEM WEARING A PLACEMENT
PROBLEM'S CLOTHES, and the board lane spent time on it as the latter.

SEVEN OF TEN CR2032 HOLDERS ARE TOO BIG FOR THIS BOARD. That is not an unlucky
pick — a 20 mm cell plus its retention on a 30 mm disc is genuinely marginal,
and it is a fact about the board's size rather than about the part. It is on
the sheet as a note.

BT1 is now the MYOUNG BS-07-A1BJ001, two pads like the 1060 so BT1.1/BT1.2 are
unchanged and the seam holds. IT IS THROUGH-HOLE, NOT SMD - a real departure
that changes how the board is assembled, recorded in the part's fields and in
a sheet note rather than absorbed. Its MPN is BS-07-A1BJ001 and it did NOT
inherit the Keystone's identity; it goes back on the lookup list as NOT
SEARCHED.

MY OWN COMMITTED BOM WAS ALREADY STALE BY THE TIME I LOOKED. It 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
Parts:
- BT1: value CR2032 3V in a holder -> CR2032 3V holder, THT; footprint Battery:BatteryHolder_Keystone_1060_1x2032 -> Battery:BatteryHolder_MYOUNG_BS-07-A1BJ001_CR2032; Courtyard (none) -> 27.41 x 6.30 mm, diagonal 28.13 mm against a 30.0 mm board; MPN Keystone 1060 -> BS-07-A1BJ001; Replaces (none) -> Keystone 1060, diagonal 39.25 mm - impossible at any positi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; Substitution basis Apple uses THREE sprung contacts with both positives sensed and no holder at all. No catalogue holder has three terminals, so this board has two and THE FIVE-REMOVALS RESET RITUAL IS NOT REPRODUCED. A real loss of function, not a simplification. -> Apple uses THREE sprung contacts with both positives sensed and no holder at all. No catalogue holder has three terminals, so this board has two and THE FIVE-REMOVALS RESET RITUAL IS NOT REPRODUCED. A real loss of function, not a simplification. THE HOLDER IS THROUGH-HOLE, not SMD like the Keystone 1060 it replaces - a real departure, because it changes how the board is assembled. It is one of only TWO parts in KiCad's Battery library whose courtyard fits a 30 mm disc (27.41 x 6.30 mm, diagonal 28.13 mm), and the other is a cell with solder tabs rather than a holder.
Other:
- note added: "THE BATTERY HOLDER IS THROUGH-HOLE AND THAT IS FORCED. SEVEN OF THE TEN CR2032 HOLDERS IN KiCad's LIBRARY ARE TOO BIG FOR THIS 30 mm BOARD - measured courtyards, all ten. The first one chosen here, a Keystone 1060, has a 39.25 mm diagonal and could not fit at any position or rotation; its courtyard was wider than the whole board, so every through-hole pad fell inside it and the board read as havi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"
- moved on the sheet: AE1, C10, C11, C12, C13, C14, C15, C16, C17, C18, C19, C20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

Commit message: correction: a5695ec's holder does not fit either, and my "independent" check reproduced the bug
a5695ec put a MYOUNG BS-07-A1BJ001 on BT1 on the strength of two surveys that
agreed its courtyard was 27.41 x 6.30 mm, diagonal 28.13, on a 30 mm board.

IT IS 27.50 x 24.42 mm, DIAGONAL 36.78. It does not fit. Neither does any
other holder.

WHY I BELIEVED IT, AND THIS IS THE ONLY PART WORTH KEEPING. I wrote in that
commit that I had "verified before changing anything, because accepting it
would have saved me the work — which is precisely when to check", and that I
had "reproduced the numbers to 0.01 mm on every row". BOTH SENTENCES ARE TRUE
AND THE CONCLUSION WAS WRONG. I did not take a second measurement. I took the
SAME measurement twice: both surveys read coordinates out of the .kicad_mod
and sampled each shape's start/mid/end POINTS.

MYOUNG's courtyard is three fp_lines and ONE fp_arc:
    (fp_arc (start 0.65 -3.15) (mid 24.564907 0) (end 0.65 3.15))
Those three points span y = -3.15..3.15, so every point-sampling parser
reports height 6.30. But the arc lies on a circle centred (12.400, 0) with
radius 12.165 and sweeps the LONG way round, through both -90 and +90 degrees,
so its true y-extent is +/-12.165. Height 24.330 plus 0.05 stroke each side =
24.43. 6.30 IS THE CHORD, NOT THE ARC.

Three confirmations that agree to 0.01 mm and are genuinely independent this
time: pcbnew's GetCourtyard().BBox() says 24.42; the board lane's closed-form
circle says 24.4298; my own closed-form, computed here from the three control
points, says 24.33 + stroke. A geometry engine and two independent
derivations, against three text parses that all said 6.30.

A GEOMETRY QUESTION MUST GO TO A GEOMETRY ENGINE. Reading coordinates out of a
file answers "what points are written down", which is a different question,
and it fails by returning a SMALLER answer rather than an error — the worst of
the three outcomes, because an empty result looks like a failure and a crash
is obvious, while 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
Parts:
- BT1: value CR2032 3V holder, THT -> CR2032 CELL - OFF-BOARD, ON 2 PADS; footprint Battery:BatteryHolder_MYOUNG_BS-07-A1BJ001_CR2032 -> Connector_PinHeader_2.54mm:PinHeader_1x02_P2.54mm_Vertical; symbol Device:Battery_Cell -> Connector_Generic:Conn_01x02; Courtyard 27.41 x 6.30 mm, diagonal 28.13 mm against a 30.0 mm board -> (none); MPN BS-07-A1BJ001 -> -; Replaces Keystone 1060, diagonal 39.25 mm - impossible at any positi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 -> (none); Substitution basis Apple uses THREE sprung contacts with both positives sensed and no holder at all. No catalogue holder has three terminals, so this board has two and THE FIVE-REMOVALS RESET RITUAL IS NOT REPRODUCED. A real loss of function, not a simplification. THE HOLDER IS THROUGH-HOLE, not SMD like the Keystone 1060 it replaces - a real departure, because it changes how the board is assembled. It is one of only TWO parts in KiCad's Battery library whose courtyard fits a 30 mm disc (27.41 x 6.30 mm, diagonal 28.13 mm), and the other is a cell with solder tabs rather than a holder. -> Apple uses THREE sprung contacts with both positives sensed and no holder at all. This board has TWO PADS and no holder either, for a different reason: NO CR2032 HOLDER IN KiCad's LIBRARY FITS A 30 mm DISC - nine of nine measurable ones are too big, measured through KiCad's own courtyard geometry. THE FIVE-REMOVALS RESET RITUAL IS NOT REPRODUCED, and now the cell is not even on the board. Both are real losses of function, stated rather than absorbed.; Why not a holder (none) -> smallest holder that fits is none; MYOUNG BS-07 diag 36.78 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; Why not a solder-tab cell (none) -> the one part that fits (Panasonic CR2032-VS1N, 21.64 mm) we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
Other:
- note added: "A HOLDER WAS SPECIFIED HERE TWICE AND BOTH WERE WRONG. A Keystone 1060 first (39.38 mm diagonal on a 30 mm board - impossible at any position, and its courtyard was wider than the whole board, so every through-hole pad fell inside it and the board read as nine placement violations when it had one part-choice problem). Then a MYOUNG BS-07, on two surveys that agreed it was 27.41 x 6.30 mm. IT IS 2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"
- note added: "THE CELL IS OFF-BOARD ON TWO PADS, AND THAT IS FORCED. NO CR2032 HOLDER IN KiCad's LIBRARY FITS A 30 mm DISC - NINE OF NINE measurable ones are too big, measured through KiCad's own courtyard geometry, and the only fitting part is a cell with solder tabs that welds the battery in permanently. A 20 mm cell plus its retention on a 30 mm disc is not marginal, it does not go. Two pads take any holder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"
- note removed: "THE BATTERY HOLDER IS THROUGH-HOLE AND THAT IS FORCED. SEVEN OF THE TEN CR2032 HOLDERS IN KiCad's LIBRARY ARE TOO BIG FOR THIS 30 mm BOARD - measured courtyards, all ten. The first one chosen here, a Keystone 1060, has a 39.25 mm diagonal and could not fit at any position or rotation; its courtyard was wider than the whole board, so every through-hole pad fell inside it and the board read as havi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"
- moved on the sheet: AE1, C1, C10, C11, C12, C13, C14, C15, C16, C17, C18, C19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
